File: Main Board/Buffered Multiple.kicad_sch (KiCad schematic)
At the start: 22 parts, among them J1 IN, J2 OUT 1, J3 OUT 2, J4 OUT 3, U3 TL074

Commit message: Upload Schematics
Other:
- note added: "Power"
- title: (none) -> KOSMO - Buffered Multiple
- moved on the sheet: C1, C2, C3, C4, C5, C6, D1, D2, D3, E1, J1, J2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
